File: Baconspoon Case and PCB/Triple Stagger Hotswap PCB (KiCad)/Switch Matrix-hotswap.kicad_sch (KiCad schematic)
At the start: 87 parts

Commit message: Add silks to PCB and flipped hotswaps to back. Add readme.
Parts:
- MX34: footprint MX_Only:MXOnly-1U-Hotswap -> MX_Only:MXOnly-1.25U-Hotswap
Changed lines of the file:
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@@
       (effects (font (size 0.508 0.508)))
     )
-    (property "Footprint" "MX_Only:MXOnly-1U-Hotswap" (at 154.305 111.125 0)
+    (property "Footprint" "MX_Only:MXOnly-1.25U-Hotswap" (at 154.305 111.125 0)
       (effects (font (size 1.524 1.524)) hide)
     )
