File: Baconspoon Case and PCB/La Cuillère - Triple Stagger Hotswap PCB (KiCad)/MCU-hotswap.kicad_sch (KiCad schematic)
At the start: 32 parts, among them J1 SM04B-SRSS-TB(LF)(SN), J2 SWD, SW1 BOOTSEL, SW2 RESET, U1 RP2040, U2 W25Q128JVS, U3 XC6206P332MR, Y1 12MHz

Commit message: Renamed PCB files and dded fabrication files.
Parts:
- added G1: Logo_Open_Hardware_Small, PCB Graphics:baconspoon-logo-15mm, symbol Graphic:Logo_Open_Hardware_Small
Changed lines of the file:
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@@
+    )
+  )
+  (symbol (lib_id "Graphic:Logo_Open_Hardware_Small") (at 259.715 32.385 0) (unit 1)
+    (in_bom no) (on_board yes) (dnp no)
+    (property "Reference" "G1" (at 259.715 25.4 0)
+      (effects (font (size 1.27 1.27)))
+    )
+    (property "Value" "Logo_Open_Hardware_Small" (at 259.715 38.1 0)
+      (effects (font (size 1.27 1.27)) hide)
+    )
+    (property "Footprint" "PCB Graphics:baconspoon-logo-15mm" (at 259.715 38.1 0)
+      (effects (font (size 1.27 1.27)))
+    )
+    (property "Datasheet" "~" (at 259.715 32.385 0)
+      (effects (font (size 1.27 1.27)) hide)
+    )
+    (property "Sim.Enable" "0" (at 259.715 32.385 0)
+      (effects (font (size 1.27 1.27)) hide)
+    )
+    (instances
+      (project "lalettre2040-tripple-stagger-hotswap-pcb"
+        (path "/0bc94950-f950-4f48-816a-6d2035325b5b/7af0d888-2a70-4b5e-b2c1-ef82dbe86c73"
+          (reference "G1") (unit 1)
+        )
+      )
+      (project "good-delivery"
+        (path "/e63e39d7-6ac0-4ffd-8aa3-1841a4541b55"
+          (reference "G2") (unit 1)
+        )
+      )
     )
   )
